File: SimpleSLIC.kicad_sch (KiCad schematic)
At the start: 16 parts, among them J1 RJ11, J2 Conn_01x02_Pin, J3 Conn_01x02_Pin, J4 Conn_01x09_Pin

Commit message: Update BOM
Parts:
- C1: DigiKey PN (none) -> 10-ECA-1EM100ICT-ND; Manufacturer (none) -> Panasonic; Manufacturer PN (none) -> ECA-1EM100I
- C2, C3, C4: DigiKey PN (none) -> BC2665CT-ND; Manufacturer (none) -> Vishay; Manufacturer PN (none) -> K104K10X7RF5UH5
- D1, D2, D3, D4: DigiKey PN (none) -> 4878-1N4004CT-ND; Manufacturer (none) -> (generic); Manufacturer PN (none) -> 1N4004
- D5: DigiKey PN (none) -> P6KE82CALFCT-ND; Manufacturer (none) -> (generic); Manufacturer PN (none) -> P6KE82CA
- D6: DigiKey PN (none) -> 1N4148-T26ACT-ND; Manufacturer (none) -> (generic); Manufacturer PN (none) -> 1N4148
- J1: DigiKey PN (none) -> WM5430-ND; Manufacturer (none) -> Molex; Manufacturer PN (none) -> 0438600003
- J2, J3: DigiKey PN (none) -> 10129378-902001BLF-ND; Manufacturer (none) -> (generic)
- J4: DigiKey PN (none) -> 10129378-909001BLF-ND; Manufacturer (none) -> (generic)
- R1: DigiKey PN (none) -> 13-CFR-25JT-52-1MCT-ND; Manufacturer (none) -> (generic); Manufacturer PN (none) -> (generic)
